Commit message: gpd working base frame workspace

File: interbotix_ros_xslocobots/interbotix_xslocobot_descriptions/urdf/locobot.urdf.xacro (robot description, xacro)
@@ -1,7 +1,7 @@
 <?xml version="1.0" ?>
 <robot name="locobot" xmlns:xacro="http://ros.org/wiki/xacro">
-  <xacro:arg name="arm_model" default=""/>
-  <xacro:arg name="robot_model" default=""/>
-  <xacro:arg name="robot_name" default=""/>
+  <xacro:arg name="arm_model" default="mobile_wx250s" />
+  <xacro:arg name="robot_model" default="mobile_wx250s" />
+  <xacro:arg name="robot_name" default="locobot" />
   <xacro:arg name="show_lidar" default="true"/>
   <xacro:arg name="show_gripper_bar" default="true"/>
@@ -21,9 +21,9 @@
     <texture filename="package://interbotix_xslocobot_descriptions/meshes/interbotix_black.png"/>
   </material>
-    <!-- ********************************** Kobuki ********************************** -->
+  <!-- ********************************** Kobuki ********************************** -->
   <link name="world"/>
-   <joint name="virtual_joint" type="fixed">
-   <parent link="world"/>
-   <child link="$(arg robot_name)_base_footprint"/>
+  <joint name="virtual_joint" type="fixed">
+    <parent link="world" />
+    <child link="$(arg robot_name)_base_footprint" />
   </joint>
   <link name="$(arg robot_name)_base_footprint"/>
@@ -42,5 +42,5 @@
     <collision>
       <origin rpy="0 0 0" xyz="0.0 0 0.05949"/>
-       <geometry>
+      <geometry>
         <mesh filename="package://interbotix_xslocobot_descriptions/meshes/locobot_meshes/locobot_main_body.dae"/>
       </geometry>
@@ -81,5 +81,5 @@
         <cylinder length="0.0206" radius="0.0352"/>
       </geometry>
-        <origin rpy="0 0 0" xyz="0 0 0"/>
+      <origin rpy="0 0 0" xyz="0 0 0" />
     </collision>
     <inertial>
@@ -207,5 +207,5 @@
     </inertial>
   </link>
-    <!-- ********************************** Bottom Plate and Arm ********************************** -->
+  <!-- ********************************** Bottom Plate and Arm ********************************** -->
   <joint name="plate" type="fixed">
     <origin rpy="0 0 0" xyz="0.0 0 0.08825"/>
@@ -237,29 +237,29 @@
     <xacro:if value="${arm_type == 'mobile_wx200'}">
       <joint name="arm_cradle" type="fixed">
-         <axis xyz="0 0 0"/>
-         <origin rpy="0 0 0" xyz="0.0215 0 0.1195"/>
-         <parent link="$(arg robot_name)_camera_tower_link"/>
-         <child link="$(arg robot_name)_arm_cradle_link"/>
+        <axis xyz="0 0 0" />
+        <origin rpy="0 0 0" xyz="0.0215 0 0.1195" />
+        <parent link="$(arg robot_name)_camera_tower_link" />
+        <child link="$(arg robot_name)_arm_cradle_link" />
       </joint>
-     <link name="$(arg robot_name)_arm_cradle_link">
-       <visual>
-         <origin rpy="0 0 0" xyz="0 0 0"/>
-         <geometry>
-           <mesh filename="package://interbotix_xslocobot_descriptions/meshes/locobot_meshes/locobot_arm_cradle.stl" scale="0.001 0.001 0.001"/>
-         </geometry>
-         <material name="interbotix_black"/>
-       </visual>
-       <collision>
-         <origin rpy="0 0 0" xyz="0 0 0"/>
-         <geometry>
-           <mesh filename="package://interbotix_xslocobot_descriptions/meshes/locobot_meshes/locobot_arm_cradle.stl" scale="0.001 0.001 0.001"/>
-         </geometry>
-       </collision>
-       <inertial>
-         <origin rpy="0 0 0" xyz="0.0014389900 0 0.0098387400"/>
-         <mass value="0.017626"/>
-         <inertia ixx="0.0000046575" ixy="0" ixz="0.0000000748" iyy="0.0000018629" iyz="0" izz="0.0000046198"/>
-       </inertial>
-     </link>
+      <link name="$(arg robot_name)_arm_cradle_link">
+        <visual>
+          <origin rpy="0 0 0" xyz="0 0 0" />
+          <geometry>
+            <mesh filename="package://interbotix_xslocobot_descriptions/meshes/locobot_meshes/locobot_arm_cradle.stl" scale="0.001 0.001 0.001" />
+          </geometry>
+          <material name="interbotix_black" />
+        </visual>
+        <collision>
+          <origin rpy="0 0 0" xyz="0 0 0" />
+          <geometry>
+            <mesh filename="package://interbotix_xslocobot_descriptions/meshes/locobot_meshes/locobot_arm_cradle.stl" scale="0.001 0.001 0.001" />
+          </geometry>
+        </collision>
+        <inertial>
+          <origin rpy="0 0 0" xyz="0.0014389900 0 0.0098387400" />
+          <mass value="0.017626" />
+          <inertia ixx="0.0000046575" ixy="0" ixz="0.0000000748" iyy="0.0000018629" iyz="0" izz="0.0000046198" />
+        </inertial>
+      </link>
     </xacro:if>
   </xacro:if>
@@ -449,8 +449,8 @@
   <link name="$(arg robot_name)_camera_optical_link"/>
   <joint name="$(arg robot_name)_camera_optical_joint" type="fixed">
-      <origin xyz="0 0 0" rpy="-${pi/2} 0 -${pi/2}"/>
-      <parent link="$(arg robot_name)_camera_link"/>
-      <child link="$(arg robot_name)_camera_optical_link"/>
-    </joint>
+    <origin xyz="0 0 0" rpy="-${pi/2} 0 -${pi/2}" />
+    <parent link="$(arg robot_name)_camera_link" />
+    <child link="$(arg robot_name)_camera_optical_link" />
+  </joint>
   <!-- ********************************** Lidar **********************************  -->
   <xacro:if value="$(arg show_lidar)">

File: interbotix_ros_xslocobots/interbotix_xslocobot_descriptions/urdf/mobile_wx250s.urdf.xacro (robot description, xacro)
@@ -1,5 +1,4 @@
 <?xml version="1.0"?>
-<robot name="mobile_wx250s"
-  xmlns:xacro="http://ros.org/wiki/xacro">
+<robot name="mobile_wx250s" xmlns:xacro="http://ros.org/wiki/xacro">
   <joint name="arm_base_link_joint" type="fixed">
     <axis xyz="0 0 0"/>

Commit message: real stack blocks works sometimes

File: interbotix_ros_xslocobots/interbotix_xslocobot_descriptions/urdf/locobot.urdf.xacro (robot description, xacro)
@@ -447,9 +447,25 @@
     </inertial>
   </link>
-  <link name="$(arg robot_name)_camera_optical_link"/>
+  <link name="$(arg robot_name)_camera_optical_link" />
   <joint name="$(arg robot_name)_camera_optical_joint" type="fixed">
-    <origin xyz="0 0 0" rpy="-${pi/2} 0 -${pi/2}" />
+    <origin xyz="0 0 0" rpy="${pi/2} 0 ${pi/2}" />
     <parent link="$(arg robot_name)_camera_link" />
+    <!-- <origin xyz="0 0 0" rpy="0 0 0" />
+    <parent link="$(arg robot_name)_base_footprint" /> -->
     <child link="$(arg robot_name)_camera_optical_link" />
+  </joint>
+  <link name="$(arg robot_name)_camera_depth_optical_link" />
+  <joint name="$(arg robot_name)_camera_depth_optical_joint" type="fixed">
+    <origin xyz="0 0 0" rpy="${pi/2} 0 ${pi/2}" />
+    <!-- <origin xyz="0 0 0" rpy="0 0 0" /> -->
+    <parent link="$(arg robot_name)_camera_link" />
+    <child link="$(arg robot_name)_camera_depth_optical_link" />
+  </joint>
+  <link name="$(arg robot_name)_camera_color_optical_link" />
+  <joint name="$(arg robot_name)_camera_color_optical_joint" type="fixed">
+    <origin xyz="0 0 0" rpy="${pi/2} 0 ${pi/2}" />
+    <!-- <origin xyz="0 0 0" rpy="0 0 0" /> -->
+    <parent link="$(arg robot_name)_camera_link" />
+    <child link="$(arg robot_name)_camera_color_optical_link" />
   </joint>
   <!-- ********************************** Lidar **********************************  -->

File: interbotix_ros_xslocobots/interbotix_xslocobot_descriptions/urdf/mobile_wx250s.urdf.xacro (robot description, xacro)
@@ -368,5 +368,6 @@
       <joint name="left_finger" type="prismatic">
         <axis xyz="0 1 0"/>
-        <limit effort="5" lower="0.015" upper="0.037" velocity="3.14"/>
+        <limit effort="5" lower="0." upper="0.5" velocity="3.14" />
+        <!-- <limit effort="5" lower="0.015" upper="0.037" velocity="3.14"/> -->
         <origin rpy="0 0 0" xyz="0 0 0"/>
         <parent link="$(arg robot_name)_fingers_link"/>
@@ -405,5 +406,6 @@
       <joint name="right_finger" type="prismatic">
         <axis xyz="0 1 0"/>
-        <limit effort="5" lower="-0.037" upper="-0.015" velocity="3.14"/>
+        <!-- <limit effort="5" lower="-0.037" upper="-0.015" velocity="3.14"/> -->
+        <limit effort="5" lower="-0.5" upper="0" velocity="3.14" />
         <origin rpy="0 0 0" xyz="0 0 0"/>
         <parent link="$(arg robot_name)_fingers_link"/>

File: interbotix_ros_xslocobots/interbotix_xslocobot_moveit/config/srdf/locobot_wx250s.srdf.xacro (robot description, xacro)
@@ -61,10 +61,10 @@
     </group_state>
     <group_state name="Sleep" group="interbotix_arm">
+        <joint name="waist" value="0" />
+        <joint name="shoulder" value="-1.1" />
         <joint name="elbow" value="1.55" />
-        <joint name="forearm_roll" value="0" />
-        <joint name="shoulder" value="-1.1" />
-        <joint name="waist" value="0" />
         <joint name="wrist_angle" value="0.5" />
         <joint name="wrist_rotate" value="0" />
+        <joint name="forearm_roll" value="0" />
     </group_state>
     <group_state name="Upright" group="interbotix_arm">
@@ -77,8 +77,8 @@
     </group_state>
     <group_state name="Home" group="interbotix_hand">
-        <joint name="left_finger" value="0.0195" />
-        <joint name="right_finger" value="-0.0195" />
-    </group_state>
-    <group_state name="Open" group="interbotix_hand">
+        <joint name="left_finger" value="0.475" />
+        <joint name="right_finger" value="-0.475" />
+    </group_state>
+    <!-- <group_state name="Open" group="interbotix_hand">
         <joint name="left_finger" value="0.037" />
         <joint name="right_finger" value="-0.037" />
@@ -87,4 +87,12 @@
         <joint name="left_finger" value="0.015" />
         <joint name="right_finger" value="-0.015" />
+    </group_state> -->
+    <group_state name="Open" group="interbotix_hand">
+        <joint name="left_finger" value="0.475" />
+        <joint name="right_finger" value="-0.475" />
+    </group_state>
+    <group_state name="Closed" group="interbotix_hand">
+        <joint name="left_finger" value="0.05" />
+        <joint name="right_finger" value="-0.05" />
     </group_state>
     <virtual_joint name="virtual_joint" type="fixed" parent_frame="world" child_link="locobot_base_footprint"/>

Commit message: changed open and close defs and optical link transforms back

File: interbotix_ros_xslocobots/interbotix_xslocobot_descriptions/urdf/locobot.urdf.xacro (robot description, xacro)
@@ -449,5 +449,5 @@
   <link name="$(arg robot_name)_camera_optical_link" />
   <joint name="$(arg robot_name)_camera_optical_joint" type="fixed">
-    <origin xyz="0 0 0" rpy="${pi/2} 0 ${pi/2}" />
+    <origin xyz="0 0 0" rpy="${-pi/2} 0 ${-pi/2}" />
     <parent link="$(arg robot_name)_camera_link" />
     <!-- <origin xyz="0 0 0" rpy="0 0 0" />
@@ -457,5 +457,5 @@
   <link name="$(arg robot_name)_camera_depth_optical_link" />
   <joint name="$(arg robot_name)_camera_depth_optical_joint" type="fixed">
-    <origin xyz="0 0 0" rpy="${pi/2} 0 ${pi/2}" />
+    <origin xyz="0 0 0" rpy="${-pi/2} 0 ${-pi/2}" />
     <!-- <origin xyz="0 0 0" rpy="0 0 0" /> -->
     <parent link="$(arg robot_name)_camera_link" />
@@ -464,5 +464,5 @@
   <link name="$(arg robot_name)_camera_color_optical_link" />
   <joint name="$(arg robot_name)_camera_color_optical_joint" type="fixed">
-    <origin xyz="0 0 0" rpy="${pi/2} 0 ${pi/2}" />
+    <origin xyz="0 0 0" rpy="${-pi/2} 0 ${-pi/2}" />
     <!-- <origin xyz="0 0 0" rpy="0 0 0" /> -->
     <parent link="$(arg robot_name)_camera_link" />

File: interbotix_ros_xslocobots/interbotix_xslocobot_moveit/config/srdf/locobot_wx250s.srdf.xacro (robot description, xacro)
@@ -80,5 +80,5 @@
         <joint name="right_finger" value="-0.475" />
     </group_state>
-    <!-- <group_state name="Open" group="interbotix_hand">
+    <group_state name="Open" group="interbotix_hand">
         <joint name="left_finger" value="0.037" />
         <joint name="right_finger" value="-0.037" />
@@ -87,6 +87,6 @@
         <joint name="left_finger" value="0.015" />
         <joint name="right_finger" value="-0.015" />
-    </group_state> -->
-    <group_state name="Open" group="interbotix_hand">
+    </group_state>
+    <!-- <group_state name="Open" group="interbotix_hand">
         <joint name="left_finger" value="0.475" />
         <joint name="right_finger" value="-0.475" />
@@ -95,5 +95,5 @@
         <joint name="left_finger" value="0.05" />
         <joint name="right_finger" value="-0.05" />
-    </group_state>
+    </group_state> -->
     <virtual_joint name="virtual_joint" type="fixed" parent_frame="world" child_link="locobot_base_footprint"/>
     <!--END EFFECTOR: Purpose: Represent information about an end effector.-->
