Commit message: Clean up gz control macros + enable diff drive

File: interbotix_ros_xslocobots/interbotix_xslocobot_descriptions/urdf/control.urdf.xacro (robot description, xacro)
@@ -1,5 +1,5 @@
 <?xml version="1.0"?>
 <robot xmlns:xacro="http://ros.org/wiki/xacro">
-  <xacro:macro name="hardware_joint_state_interface">
+  <xacro:macro name="hardware_interface">
     <hardware>
       <!-- If we are using the actual, physical robot -->
@@ -155,5 +155,5 @@
       'kobuki' -->
   </xacro:macro>
-  <xacro:macro name="gz_controller_manager">
+  <xacro:macro name="gz_control_provider">
     <xacro:if value="${hardware_type == 'gz_classic'}">
       <plugin name="gazebo_ros2_control" filename="libgazebo_ros2_control.so">
@@ -170,7 +170,5 @@
       <plugin filename="ign_ros2_control-system"
         name="ign_ros2_control::IgnitionROS2ControlPlugin">
-        <!-- <ros>
-          <namespace>/$(arg robot_name)</namespace>
-        </ros> -->
+        <robot_param>robot_description</robot_param>
         <parameters>
           $(find interbotix_xslocobot_sim)/config/${base_type}_version/${

File: interbotix_ros_xslocobots/interbotix_xslocobot_descriptions/urdf/locobot.urdf.xacro (robot description, xacro)
@@ -336,16 +336,28 @@
   <xacro:include filename="$(find interbotix_xslocobot_descriptions)/urdf/control.urdf.xacro" />
   <gazebo>
-    <xacro:gz_controller_manager />
+    <!-- Loads simulated hardware interface. -->
+    <xacro:gz_control_provider />
+    <!-- Loads simulated sensors. -->
     <plugin
       filename="ignition-gazebo-sensors-system"
       name="ignition::gazebo::systems::Sensors">
-      <ignition_frame_id>/${robot_name}_base_footprint</ignition_frame_id>
-      <ros>
-        <namespace></namespace>
-      </ros>
     </plugin>
+    <!-- <plugin
+      filename="libignition-gazebo-diff-drive-system.so"
+      name="ignition::gazebo::systems::DiffDrive">
+      <left_joint>wheel_left_joint</left_joint>
+      <right_joint>wheel_right_joint</right_joint>
+      <wheel_separation>0.230</wheel_separation>
+      <wheel_radius>0.035</wheel_radius>
+      <odom_publish_frequency>62</odom_publish_frequency>
+      <topic>cmd_vel</topic>
+    </plugin> -->
+    <!-- <plugin filename="ignition-gazebo-joint-state-publisher-system"
+      name="ignition::gazebo::systems::JointStatePublisher" /> -->
   </gazebo>
+  <!-- Defines hardware interface. -->
   <ros2_control name="SystemControl" type="system">
-    <xacro:hardware_joint_state_interface />
+    <xacro:hardware_interface />
+    <!-- TODO:(speralta): Move pan_and_tilt sensors here? -->
   </ros2_control>
 </robot>
