Commit message: Enable octomap from RGBD sensor + fix tf tree root

File: interbotix_ros_xslocobots/interbotix_xslocobot_descriptions/urdf/kobuki_version/locobot_kobuki.urdf.xacro (robot description, xacro)
@@ -38,11 +38,4 @@
     # POSSIBILITY OF SUCH DAMAGE.
   -->
-  <link name="world"/>
-  <joint name="virtual_joint" type="fixed">
-    <parent
-      link="world"/>
-    <child
-      link="${robot_name}_base_footprint"/>
-  </joint>
   <link name="${robot_name}_base_footprint"/>
   <joint name="base_joint" type="fixed">

File: interbotix_ros_xslocobots/interbotix_xslocobot_moveit/config/srdf/locobot_wx250s.srdf.xacro (robot description, xacro)
@@ -71,6 +71,7 @@
         <joint name="right_finger" value="-0.015" />
     </group_state>
-    <virtual_joint name="virtual_joint" child_link="${robot_name}_base_footprint"
-        parent_frame="world" type="fixed" />
+    <!-- Define how the robot moves in its environment, i.e., connection to robot's root link -->
+    <virtual_joint name="virtual_joint" type="planar" parent_frame="odom"
+        child_link="locobot_base_footprint" /> <!-- type can be planar, floating or fixed -->
     <!--END EFFECTOR - Purpose - Represent information about an end effector.-->
     <end_effector name="interbotix_gripper" parent_link="${robot_name}_ee_gripper_link"

Commit message: ns urdf links

File: interbotix_ros_xslocobots/interbotix_xslocobot_descriptions/urdf/kobuki_version/locobot_kobuki.urdf.xacro (robot description, xacro)
@@ -376,10 +376,10 @@
       <wheelAcceleration>0</wheelAcceleration>
       <commandTopic>mobile_base/commands/velocity</commandTopic>
-      <odometryTopic>mobile_base/odom</odometryTopic>
-      <odometryFrame>$(arg robot_name)/odom</odometryFrame>
+      <odometryTopic>$(arg robot_name)/odom</odometryTopic>
+      <odometryFrame>world</odometryFrame>
       <robotBaseFrame>$(arg robot_name)/base_footprint</robotBaseFrame>
       <publishWheelJointState>true</publishWheelJointState>
       <rosDebugLevel>na</rosDebugLevel>
-      <publishWheelTF>false</publishWheelTF>
+      <publishWheelTF>true</publishWheelTF>
       <publishOdomTF>true</publishOdomTF>
       <odometrySource>world</odometrySource>

File: interbotix_ros_xslocobots/interbotix_xslocobot_descriptions/urdf/locobot.urdf.xacro (robot description, xacro)
@@ -25,4 +25,9 @@
   <xacro:include filename="$(find interbotix_xslocobot_descriptions)/urdf/camera_tower.urdf.xacro" />
   <xacro:include filename="$(find interbotix_xslocobot_descriptions)/urdf/pan_and_tilt.urdf.xacro" />
+  <link name="world"/>
+  <joint name="virtual_joint" type="fixed">
+    <parent link="world" />
+    <child link="$(arg robot_name)/base_footprint" />
+  </joint>
   <link name="$(arg robot_name)/base_footprint"/>
   <xacro:if value="${arm_type == 'mobile_wx250s'}">

File: interbotix_ros_xslocobots/interbotix_xslocobot_moveit/config/srdf/locobot_wx250s.srdf.xacro (robot description, xacro)
@@ -68,4 +68,5 @@
         <joint name="right_finger" value="-0.015" />
     </group_state>
+     <virtual_joint name="virtual_joint" type="fixed" parent_frame="world" child_link="$(arg robot_name)/base_footprint" />
     <!--END EFFECTOR: Purpose: Represent information about an end effector.-->
     <end_effector name="interbotix_gripper" parent_link="$(arg robot_name)/ee_gripper_link" group="interbotix_gripper" />
