Commit message: stack blocks working docker vnc

File: interbotix_ros_xslocobots/interbotix_xslocobot_descriptions/urdf/arms/mobile_wx250s.urdf.xacro (robot description, xacro)
@@ -3,31 +3,33 @@
   <xacro:property name="dof"
     value="6"
-    scope="global"/>
-  <xacro:property name="mesh_directory"             value="package://interbotix_xslocobot_descriptions/meshes/${arm_type}_meshes"/>
-  <xacro:property name="urdf_loc"                   value="$(arg external_urdf_loc)"/>
-  <xacro:property name="hardware_type"              value="$(arg hardware_type)"/>
-  <xacro:property name="pi_offset"                  value="0.00001"/>
-  <!-- <xacro:include filename="$(find interbotix_xslocobot_descriptions)/urdf/arms/arm_control.urdf.xacro"/> -->
-  <xacro:include filename="$(find interbotix_xslocobot_descriptions)/urdf/arms/ar_tag.urdf.xacro"/>
+    scope="global" />
+  <xacro:property name="mesh_directory"
+    value="package://interbotix_xslocobot_descriptions/meshes/${arm_type}_meshes" />
+  <xacro:property name="urdf_loc" value="$(arg external_urdf_loc)" />
+  <xacro:property name="hardware_type" value="$(arg hardware_type)" />
+  <xacro:property name="pi_offset" value="0.00001" />
+  <!-- <xacro:include filename="$(find
+  interbotix_xslocobot_descriptions)/urdf/arms/arm_control.urdf.xacro"/> -->
+  <xacro:include filename="$(find interbotix_xslocobot_descriptions)/urdf/arms/ar_tag.urdf.xacro" />
   <link name="${robot_name}_arm_base_link">
     <visual>
       <origin
         rpy="${pi/2} 0 ${pi/2}"
-        xyz="-0.095773 0 -0.10565023"/>
+        xyz="-0.095773 0 -0.10565023" />
       <geometry>
         <mesh
           filename="${mesh_directory}/base.stl"
-          scale="0.001 0.001 0.001"/>
-      </geometry>
-      <material name="interbotix_black"/>
+          scale="0.001 0.001 0.001" />
+      </geometry>
+      <material name="interbotix_black" />
     </visual>
     <collision>
       <origin
         rpy="${pi/2} 0 ${pi/2}"
-        xyz="-0.095773 0 -0.10565023"/>
+        xyz="-0.095773 0 -0.10565023" />
       <geometry>
         <mesh
           filename="${mesh_directory}/base.stl"
-          scale="0.001 0.001 0.001"/>
+          scale="0.001 0.001 0.001" />
       </geometry>
     </collision>
@@ -35,6 +37,6 @@
       <origin
         rpy="${pi/2} 0 ${pi/2}"
-        xyz="-0.0001350000 -0.0000266286 0.0338755000"/>
-      <mass value="0.379673"/>
+        xyz="-0.0001350000 -0.0000266286 0.0338755000" />
+      <mass value="0.379673" />
       <inertia
         ixx="0.0004351000"
@@ -43,24 +45,24 @@
         ixy="0.0000000707"
         ixz="0.0000000266"
-        iyz="-0.0000022881"/>
+        iyz="-0.0000022881" />
     </inertial>
   </link>
   <joint name="waist" type="revolute">
-    <axis xyz="0 0 1"/>
+    <axis xyz="0 0 1" />
     <limit
       effort="${waist_limit_effort}"
       lower="${waist_limit_lower}"
       upper="${waist_limit_upper}"
-      velocity="${waist_limit_vel}"/>
+      velocity="${waist_limit_vel}" />
     <origin
       rpy="0 0 0"
-      xyz="0 0 0.066175"/>
+      xyz="0 0 0.066175" />
     <parent
-      link="${robot_name}_arm_base_link"/>
+      link="${robot_name}_arm_base_link" />
     <child
-      link="${robot_name}_shoulder_link"/>
+      link="${robot_name}_shoulder_link" />
     <dynamics
       friction="0.1"
-      damping="0.1"/>
+      damping="0.1" />
   </joint>
   <link name="${robot_name}_shoulder_link">
@@ -68,20 +70,20 @@
       <origin
         rpy="0 0 ${pi/2}"
-        xyz="0 0 -0.003"/>
+        xyz="0 0 -0.003" />
       <geometry>
         <mesh
           filename="${mesh_directory}/shoulder.stl"
-          scale="0.001 0.001 0.001"/>
-      </geometry>
-      <material name="interbotix_black"/>
+          scale="0.001 0.001 0.001" />
+      </geometry>
+      <material name="interbotix_black" />
     </visual>
     <collision>
       <origin
         rpy="0 0 ${pi/2}"
-        xyz="0 0 -0.003"/>
+        xyz="0 0 -0.003" />
       <geometry>
         <mesh
           filename="${mesh_directory}/shoulder.stl"
-          scale="0.001 0.001 0.001"/>
+          scale="0.001 0.001 0.001" />
       </geometry>
     </collision>
@@ -89,6 +91,6 @@
       <origin
         rpy="0 0 ${pi/2}"
-        xyz="0.0000223482 0.0000414609 0.0066287000"/>
-      <mass value="0.480879"/>
+        xyz="0.0000223482 0.0000414609 0.0066287000" />
+      <mass value="0.480879" />
       <inertia
         ixx="0.0003790000"
@@ -97,24 +99,24 @@
         ixy="0.0000000022"
         ixz="-0.0000003561"
-        iyz="0.0000012245"/>
+        iyz="0.0000012245" />
     </inertial>
   </link>
   <joint name="shoulder" type="revolute">
-    <axis xyz="0 1 0"/>
+    <axis xyz="0 1 0" />
     <limit
       effort="${shoulder_limit_effort}"
       lower="${shoulder_limit_lower}"
       upper="${shoulder_limit_upper}"
-      velocity="${shoulder_limit_vel}"/>
+      velocity="${shoulder_limit_vel}" />
     <origin
       rpy="0 0 0"
-      xyz="0 0 0.03865"/>
+      xyz="0 0 0.03865" />
     <parent
-      link="${robot_name}_shoulder_link"/>
+      link="${robot_name}_shoulder_link" />
     <child
-      link="${robot_name}_upper_arm_link"/>
+      link="${robot_name}_upper_arm_link" />
     <dynamics
       friction="0.1"
-      damping="0.1"/>
+      damping="0.1" />
   </joint>
   <link name="${robot_name}_upper_arm_link">
@@ -122,20 +124,20 @@
       <origin
         rpy="0 0 ${pi/2}"
-        xyz="0 0 0"/>
+        xyz="0 0 0" />
       <geometry>
         <mesh
           filename="${mesh_directory}/upper_arm.stl"
-          scale="0.001 0.001 0.001"/>
-      </geometry>
-      <material name="interbotix_black"/>
+          scale="0.001 0.001 0.001" />
+      </geometry>
+      <material name="interbotix_black" />
     </visual>
     <collision>
       <origin
         rpy="0 0 ${pi/2}"
-        xyz="0 0 0"/>
+        xyz="0 0 0" />
       <geometry>
         <mesh
           filename="${mesh_directory}/upper_arm.stl"
-          scale="0.001 0.001 0.001"/>
+          scale="0.001 0.001 0.001" />
       </geometry>
     </collision>
@@ -143,6 +145,6 @@
       <origin
         rpy="0 0 ${pi/2}"
-        xyz="0.0171605000 0.0000002725 0.1913230000"/>
-      <mass value="0.430811"/>
+        xyz="0.0171605000 0.0000002725 0.1913230000" />
+      <mass value="0.430811" />
       <inertia
         ixx="0.0034630000"
@@ -151,24 +153,24 @@
         ixy="-0.0000000001"
         ixz="-0.0000000002"
-        iyz="0.0004272000"/>
+        iyz="0.0004272000" />
     </inertial>
   </link>
   <joint name="elbow" type="revolute">
-    <axis xyz="0 1 0"/>
+    <axis xyz="0 1 0" />
     <limit
       effort="${elbow_limit_effort}"
       lower="${elbow_limit_lower}"
       upper="${elbow_limit_upper}"
-      velocity="${elbow_limit_vel}"/>
+      velocity="${elbow_limit_vel}" />
     <origin
       rpy="0 0 0"
-      xyz="0.04975 0 0.25"/>
+      xyz="0.04975 0 0.25" />
     <parent
-      link="${robot_name}_upper_arm_link"/>
+      link="${robot_name}_upper_arm_link" />
     <child
-      link="${robot_name}_upper_forearm_link"/>
+      link="${robot_name}_upper_forearm_link" />
     <dynamics
       friction="0.1"
-      damping="0.1"/>
+      damping="0.1" />
   </joint>
   <link name="${robot_name}_upper_forearm_link">
@@ -176,20 +178,20 @@
       <origin
         rpy="0 0 0"
-        xyz="0 0 0"/>
+        xyz="0 0 0" />
       <geometry>
         <mesh
           filename="${mesh_directory}/upper_forearm.stl"
-          scale="0.001 0.001 0.001"/>
-      </geometry>
-      <material name="interbotix_black"/>
+          scale="0.001 0.001 0.001" />
+      </geometry>
+      <material name="interbotix_black" />
     </visual>
     <collision>
       <origin
         rpy="0 0 0"
-        xyz="0 0 0"/>
+        xyz="0 0 0" />
       <geometry>
         <mesh
           filename="${mesh_directory}/upper_forearm.stl"
-          scale="0.001 0.001 0.001"/>
+          scale="0.001 0.001 0.001" />
       </geometry>
     </collision>
@@ -197,6 +199,6 @@
       <origin
         rpy="0 0 0"
-        xyz="0.1079630000 0.0001158760 0"/>
-      <mass value="0.234589"/>
+        xyz="0.1079630000 0.0001158760 0" />
+      <mass value="0.234589" />
       <inertia
         ixx="0.0000397100"
@@ -205,22 +207,22 @@
         ixy="0.0000023528"
         ixz="0"
-        iyz="0"/>
+        iyz="0" />
     </inertial>
   </link>
   <joint name="forearm_roll" type="revolute">
-    <axis xyz="1 0 0"/>
+    <axis xyz="1 0 0" />
     <limit
       effort="${forearm_roll_limit_effort}"
       lower="${forearm_roll_limit_lower}"
       upper="${forearm_roll_limit_upper}"
-      velocity="${forearm_roll_limit_vel}"/>
-    <origin rpy="0 0 0" xyz="0.175 0 0"/>
+      velocity="${forearm_roll_limit_vel}" />
+    <origin rpy="0 0 0" xyz="0.175 0 0" />
     <parent
-      link="${robot_name}_upper_forearm_link"/>
+      link="${robot_name}_upper_forearm_link" />
     <child
-      link="${robot_name}_lower_forearm_link"/>
+      link="${robot_name}_lower_forearm_link" />
     <dynamics
       friction="0.1"
-      damping="0.1"/>
+      damping="0.1" />
   </joint>
   <link name="${robot_name}_lower_forearm_link">
@@ -228,20 +230,20 @@
       <origin
         rpy="${pi} 0 0"
-        xyz="0 0 0"/>
+        xyz="0 0 0" />
       <geometry>
         <mesh
           filename="${mesh_directory}/lower_forearm.stl"
-          scale="0.001 0.001 0.001"/>
-      </geometry>
-      <material name="interbotix_black"/>
+          scale="0.001 0.001 0.001" />
+      </geometry>
+      <material name="interbotix_black" />
     </visual>
     <collision>
       <origin
         rpy="${pi} 0 0"
-        xyz="0 0 0"/>
+        xyz="0 0 0" />
       <geometry>
         <mesh
           filename="${mesh_directory}/lower_forearm.stl"
-          scale="0.001 0.001 0.001"/>
+          scale="0.001 0.001 0.001" />
       </geometry>
     </collision>
@@ -249,6 +251,6 @@
       <origin
         rpy="${pi} 0 0"
-        xyz="0.0374395000 0.0052225200 0"/>
-      <mass value="0.220991"/>
+        xyz="0.0374395000 0.0052225200 0" />
+      <mass value="0.220991" />
       <inertia
         ixx="0.0000636900"
@@ -257,24 +259,24 @@
         ixy="-0.0000229200"
         ixz="0"
-        iyz="0"/>
+        iyz="0" />
     </inertial>
   </link>
- <joint name="wrist_angle" type="revolute">
-    <axis xyz="0 1 0"/>
+  <joint name="wrist_angle" type="revolute">
+    <axis xyz="0 1 0" />
     <limit
       effort="${wrist_angle_limit_effort}"
       lower="${wrist_angle_limit_lower}"
       upper="${wrist_angle_limit_upper}"
-      velocity="${wrist_angle_limit_vel}"/>
+      velocity="${wrist_angle_limit_vel}" />
     <origin
       rpy="0 0 0"
-      xyz="0.075 0 0"/>
+      xyz="0.075 0 0" />
     <parent
-      link="${robot_name}_lower_forearm_link"/>
+      link="${robot_name}_lower_forearm_link" />
     <child
-      link="${robot_name}_wrist_link"/>
+      link="${robot_name}_wrist_link" />
     <dynamics
       friction="0.1"
-      damping="0.1"/>
+      damping="0.1" />
   </joint>
   <link name="${robot_name}_wrist_link">
@@ -282,20 +284,20 @@
       <origin
         rpy="0 0 ${pi/2}"
-        xyz="0 0 0"/>
+        xyz="0 0 0" />
       <geometry>
         <mesh
           filename="${mesh_directory}/wrist.stl"
-          scale="0.001 0.001 0.001"/>
-      </geometry>
-      <material name="interbotix_black"/>
+          scale="0.001 0.001 0.001" />
+      </geometry>
+      <material name="interbotix_black" />
     </visual>
     <collision>
       <origin
         rpy="0 0 ${pi/2}"
-        xyz="0 0 0"/>
+        xyz="0 0 0" />
       <geometry>
         <mesh
           filename="${mesh_directory}/wrist.stl"
-          scale="0.001 0.001 0.001"/>
+          scale="0.001 0.001 0.001" />
       </geometry>
     </collision>
@@ -303,6 +305,6 @@
       <origin
         rpy="0 0 ${pi/2}"
-        xyz="0.0423600000 -0.0000106630 0.0105770000"/>
-      <mass value="0.084957"/>
+        xyz="0.0423600000 -0.0000106630 0.0105770000" />
+      <mass value="0.084957" />
       <inertia
         ixx="0.0000308200"
@@ -311,5 +313,5 @@
         ixy="0.0000000191"
         ixz="0.0000000023"
-        iyz="0.0000025481"/>
+        iyz="0.0000025481" />
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
File: interbotix_ros_xslocobots/interbotix_xslocobot_descriptions/urdf/control.urdf.xacro (robot description, xacro)
@@ -24,10 +24,10 @@
       </xacro:if>
     </hardware>
-  <joint name="waist">
+    <joint name="waist">
       <command_interface name="position">
         <param name="min">"${waist_limit_lower}"</param>
         <param name="max">"${waist_limit_upper}"</param>
       </command_interface>
-      <state_interface name="position"/>
+      <state_interface name="position" />
       <param name="initial_position">0.00</param>
     </joint>
@@ -37,5 +37,5 @@
         <param name="max">"${shoulder_limit_upper}"</param>
       </command_interface>
-      <state_interface name="position"/>
+      <state_interface name="position" />
       <param name="initial_position">0.00</param>
     </joint>
@@ -45,5 +45,5 @@
         <param name="max">"${elbow_limit_upper}"</param>
       </command_interface>
-      <state_interface name="position"/>
+      <state_interface name="position" />
       <param name="initial_position">0.00</param>
     </joint>
@@ -54,5 +54,5 @@
           <param name="max">"${forearm_roll_limit_upper}"</param>
         </command_interface>
-        <state_interface name="position"/>
+        <state_interface name="position" />
         <param name="initial_position">0.00</param>
       </joint>
@@ -63,5 +63,5 @@
         <param name="max">"${wrist_angle_limit_upper}"</param>
       </command_interface>
-      <state_interface name="position"/>
+      <state_interface name="position" />
       <param name="initial_position">0.00</param>
     </joint>
@@ -72,5 +72,5 @@
           <param name="max">"${wrist_rotate_limit_upper}"</param>
         </command_interface>
-        <state_interface name="position"/>
+        <state_interface name="position" />
         <param name="initial_position">0.00</param>
       </joint>
@@ -79,6 +79,6 @@
       <xacro:if value="${hardware_type in ('fake', 'gz_classic', 'gz_ignition')}">
         <joint name="gripper">
-          <command_interface name="position"/>
-          <state_interface name="position"/>
+          <command_interface name="position" />
+          <state_interface name="position" />
         </joint>
       </xacro:if>
@@ -86,8 +86,8 @@
         <joint name="left_finger">
           <command_interface name="position">
-            <param name="min">"${finger_limit_lower}"</param>
-            <param name="max">"${-finger_limit_lower}"</param>
+            <param name="min">${finger_limit_lower}</param>
+            <param name="max">${finger_limit_upper}</param>
           </command_interface>
-          <state_interface name="position"/>
+          <state_interface name="position" />
           <param name="initial_position">0.0195</param>
         </joint>
@@ -97,86 +97,86 @@
             <param name="multiplier">1</param> -->
             <command_interface name="position">
-              <param name="min">"${-finger_limit_lower}"</param>
-              <param name="max">"${finger_limit_lower}"</param>
+              <param name="min">${-finger_limit_upper}</param>
+              <param name="max">${-finger_limit_lower}"</param>
             </command_interface>
-            <state_interface name="position"/>
-            <param name="initial_position">0.0195</param>
+            <state_interface name="position" />
+            <param name="initial_position">-0.0195</param>
           </joint>
         </xacro:if>
       </xacro:if>
     </xacro:if>
-      <joint name="pan">
+    <joint name="pan">
+      <command_interface name="position" />
+      <state_interface name="position" />
+      <param name="initial_position">0.0</param>  <!-- initial position for the GenericSystem -->
+    </joint>
+    <joint name="tilt">
+      <command_interface name="position" />
+      <state_interface name="position" />
+      <param name="initial_position">0.0</param>  <!-- initial position for the GenericSystem -->
+    </joint>
+    <xacro:if value="${base_type == 'create3'}">
+      <joint name="wheel_drop_left_joint">
         <command_interface name="position" />
         <state_interface name="position" />
         <param name="initial_position">0.0</param>  <!-- initial position for the GenericSystem -->
       </joint>
-      <joint name="tilt">
+      <joint name="wheel_drop_right_joint">
         <command_interface name="position" />
         <state_interface name="position" />
         <param name="initial_position">0.0</param>  <!-- initial position for the GenericSystem -->
       </joint>
-      <xacro:if value="${base_type == 'create3'}">
-        <joint name="wheel_drop_left_joint">
-          <command_interface name="position" />
-          <state_interface name="position" />
-          <param name="initial_position">0.0</param>  <!-- initial position for the GenericSystem -->
-        </joint>
-        <joint name="wheel_drop_right_joint">
-          <command_interface name="position" />
-          <state_interface name="position" />
-          <param name="initial_position">0.0</param>  <!-- initial position for the GenericSystem -->
-        </joint>
-        <joint name="left_wheel_joint">
-          <command_interface name="position" />
-          <command_interface name="velocity" />
-          <state_interface name="position" />
-          <state_interface name="velocity" />
-          <param name="initial_position">0.0</param>  <!-- initial position for the GenericSystem -->
-        </joint>
-        <joint name="right_wheel_joint">
-          <command_interface name="position" />
-          <command_interface name="velocity" />
-          <state_interface name="position" />
-          <state_interface name="velocity" />
-          <param name="initial_position">0.0</param>  <!-- initial position for the GenericSystem -->
-        </joint>
-      </xacro:if> <!-- base_type
+      <joint name="left_wheel_joint">
+        <command_interface name="position" />
+        <command_interface name="velocity" />
+        <state_interface name="position" />
+        <state_interface name="velocity" />
+        <param name="initial_position">0.0</param>  <!-- initial position for the GenericSystem -->
+      </joint>
+      <joint name="right_wheel_joint">
+        <command_interface name="position" />
+        <command_interface name="velocity" />
+        <state_interface name="position" />
+        <state_interface name="velocity" />
+        <param name="initial_position">0.0</param>  <!-- initial position for the GenericSystem -->
+      </joint>
+    </xacro:if> <!-- base_type
     =='create3' -->
-      <xacro:if value="${base_type == 'kobuki'}">
-        <joint name="wheel_left_joint">
-          <command_interface name="velocity" />
-          <state_interface name="position" />
-        </joint>
-        <joint name="wheel_right_joint">
-          <command_interface name="velocity" />
-          <state_interface name="position" />
-        </joint>
-      </xacro:if> <!-- base_type ==
+    <xacro:if value="${base_type == 'kobuki'}">
+      <joint name="wheel_left_joint">
+        <command_interface name="velocity" />
+        <state_interface name="position" />
+      </joint>
+      <joint name="wheel_right_joint">
+        <command_interface name="velocity" />
+        <state_interface name="position" />
+      </joint>
+    </xacro:if> <!-- base_type ==
       'kobuki' -->
-</xacro:macro>
-<xacro:macro name="gz_controller_manager">
-      <xacro:if value="${hardware_type == 'gz_classic'}">
-        <plugin name="gazebo_ros2_control" filename="libgazebo_ros2_control.so">
-          <ros>
-            <namespace>/${robot_name}</namespace>
-          </ros>
-          <robot_param>robot_description</robot_param>
-          <robot_param_node>robot_state_publisher</robot_param_node>
-          <parameters> $(find interbotix_xslocobot_sim)/config/${base_type}_version/${
-            robot_model}_controllers.yaml </parameters>
-        </plugin>
-      </xacro:if>
-      <xacro:if value="${hardware_type == 'gz_ignition'}">
-        <plugin filename="ign_ros2_control-system"
-          name="ign_ros2_control::IgnitionROS2ControlPlugin">
-          <!-- <ros>
+  </xacro:macro>
+  <xacro:macro name="gz_controller_manager">
+    <xacro:if value="${hardware_type == 'gz_classic'}">
+      <plugin name="gazebo_ros2_control" filename="libgazebo_ros2_control.so">
+        <ros>
+          <namespace>/${robot_name}</namespace>
+        </ros>
+        <robot_param>robot_description</robot_param>
+        <robot_param_node>robot_state_publisher</robot_param_node>
+        <parameters> $(find interbotix_xslocobot_sim)/config/${base_type}_version/${
+          robot_model}_controllers.yaml </parameters>
+      </plugin>
+    </xacro:if>
+    <xacro:if value="${hardware_type == 'gz_ignition'}">
+      <plugin filename="ign_ros2_control-system"
+        name="ign_ros2_control::IgnitionROS2ControlPlugin">
+        <!-- <ros>
           <namespace>/$(arg robot_name)</namespace>
         </ros> -->
-          <parameters>
-            $(find interbotix_xslocobot_sim)/config/${base_type}_version/${
-            robot_model}_controllers.yaml
-          </parameters>
-        </plugin>
-      </xacro:if>
+        <parameters>
+          $(find interbotix_xslocobot_sim)/config/${base_type}_version/${
+          robot_model}_controllers.yaml
+        </parameters>
+      </plugin>
+    </xacro:if>
   </xacro:macro>
 </robot>
