Commit message: stack blocks working docker vnc

File: interbotix_ros_xslocobots/interbotix_xslocobot_descriptions/urdf/lidar.urdf.xacro (robot description, xacro)
@@ -1,11 +1,11 @@
-<?xml version="1.0" ?>
+<?xml version="1.0"?>
 <robot xmlns:xacro="http://ros.org/wiki/xacro">
   <xacro:macro name="lidar" params="*origin">
     <joint name="lidar_tower" type="fixed">
-      <xacro:insert_block name="origin"/>
+      <xacro:insert_block name="origin" />
       <parent
-        link="${robot_name}_camera_tower_link"/>
+        link="${robot_name}_camera_tower_link" />
       <child
-        link="${robot_name}_lidar_tower_link"/>
+        link="${robot_name}_lidar_tower_link" />
     </joint>
     <link name="${robot_name}_lidar_tower_link">
@@ -13,20 +13,20 @@
         <origin
           rpy="0 0 0"
-          xyz="0 0 0"/>
+          xyz="0 0 0" />
         <geometry>
           <mesh
             filename="package://interbotix_xslocobot_descriptions/meshes/locobot_meshes/locobot_lidar_tower.stl"
-            scale="0.001 0.001 0.001"/>
+            scale="0.001 0.001 0.001" />
         </geometry>
-        <material name="interbotix_black"/>
+        <material name="interbotix_black" />
       </visual>
       <collision>
         <origin
           rpy="0 0 0"
-          xyz="0 0 0"/>
+          xyz="0 0 0" />
         <geometry>
           <mesh
             filename="package://interbotix_xslocobot_descriptions/meshes/locobot_meshes/locobot_lidar_tower_simple.stl"
-            scale="0.001 0.001 0.001"/>
+            scale="0.001 0.001 0.001" />
         </geometry>
       </collision>
@@ -34,6 +34,6 @@
         <origin
           rpy="0 0 0"
-          xyz="-0.0074822400 -0.0000196881 0.0507957000"/>
-        <mass value="0.155485"/>
+          xyz="-0.0074822400 -0.0000196881 0.0507957000" />
+        <mass value="0.155485" />
         <inertia
           ixx="0.0007642000"
@@ -42,5 +42,5 @@
           iyy="0.0001285000"
           iyz="0.0000000354"
-          izz="0.0007840000"/>
+          izz="0.0007840000" />
       </inertial>
     </link>
@@ -48,9 +48,9 @@
       <origin
         rpy="0 0 ${pi}"
-        xyz="0 0 0.09425"/>
+        xyz="0 0 0.09425" />
       <parent
-        link="${robot_name}_lidar_tower_link"/>
+        link="${robot_name}_lidar_tower_link" />
       <child
-        link="${robot_name}_laser_frame_link"/>
+        link="${robot_name}_laser_frame_link" />
     </joint>
     <link name="${robot_name}_laser_frame_link">
@@ -58,20 +58,20 @@
         <origin
           rpy="0 0 0"
-          xyz="0 0 0"/>
+          xyz="0 0 0" />
         <geometry>
           <mesh
             filename="package://interbotix_xslocobot_descriptions/meshes/locobot_meshes/locobot_lidar.stl"
-            scale="0.001 0.001 0.001"/>
+            scale="0.001 0.001 0.001" />
         </geometry>
-        <material name="interbotix_black"/>
+        <material name="interbotix_black" />
       </visual>
       <collision>
         <origin
           rpy="0 0 0"
-          xyz="0 0 -0.0091"/>
+          xyz="0 0 -0.0091" />
         <geometry>
           <cylinder
             length="0.0408"
-            radius="0.03785"/>
+            radius="0.03785" />
         </geometry>
       </collision>
@@ -79,6 +79,6 @@
         <origin
           rpy="0 0 0"
-          xyz="0.0007379970 0 -0.0103809000"/>
-        <mass value="0.196"/>
+          xyz="0.0007379970 0 -0.0103809000" />
+        <mass value="0.196" />
         <inertia
           ixx="0.0000907500"
@@ -87,5 +87,5 @@
           iyy="0.0000877600"
           iyz="0"
-          izz="0.0001268000"/>
+          izz="0.0001268000" />
       </inertial>
     </link>
@@ -101,8 +101,9 @@
     <gazebo reference="${robot_name}_laser_frame_link">
       <material>Gazebo/DarkGrey</material>
-      <sensor type="ray" name="rplidar">
+      <sensor type="gpu_lidar" name="rplidar">
         <always_on>true</always_on>
         <visualize>false</visualize>
         <pose>0 0 0 0 0 0</pose>
+        <topic>/scan</topic>
         <update_rate>30</update_rate>
         <ray>
@@ -127,13 +128,13 @@
         </ray>
         <xacro:if value="${hardware_type == 'gz_classic'}">
-        <plugin name="gazebo_ros_head_rplidar_controller" filename="libgazebo_ros_ray_sensor.so">
-          <!-- <ros>
+          <plugin name="gazebo_ros_head_rplidar_controller" filename="libgazebo_ros_ray_sensor.so">
+            <!-- <ros>
             <remapping>~/out:=${robot_name}/scan</remapping>
           </ros> -->
-          <output_type>sensor_msgs/LaserScan</output_type>
-          <frame_name>${robot_name}_laser_frame_link</frame_name>
-        </plugin>
+            <output_type>sensor_msgs/LaserScan</output_type>
+            <frame_name>${robot_name}_laser_frame_link</frame_name>
+          </plugin>
         </xacro:if>
-        <xacro:if value="${hardware_type == 'gz_ignition'}">
+        <!-- <xacro:if value="${hardware_type == 'gz_ignition'}">
           <plugin
           filename="libignition-gazebo-sensors-system.so"
@@ -143,5 +144,5 @@
           <frame_name>${robot_name}_laser_frame_link</frame_name>
         </plugin>
-        </xacro:if>
+        </xacro:if> -->
       </sensor>
     </gazebo>

File: interbotix_ros_xslocobots/interbotix_xslocobot_descriptions/urdf/pan_and_tilt.urdf.xacro (robot description, xacro)
@@ -1,20 +1,20 @@
-<?xml version="1.0" ?>
+<?xml version="1.0"?>
 <robot xmlns:xacro="http://ros.org/wiki/xacro">
   <xacro:macro name="pan_and_tilt" params="*origin">
     <joint name="pan" type="revolute">
-      <axis xyz="0 0 1"/>
+      <axis xyz="0 0 1" />
       <limit
         effort="2"
         lower="${-pi/2}"
         upper="${pi/2}"
-        velocity="${pi}"/>
-      <xacro:insert_block name="origin"/>
+        velocity="${pi}" />
+      <xacro:insert_block name="origin" />
       <parent
-        link="${robot_name}_camera_tower_link"/>
+        link="${robot_name}_camera_tower_link" />
       <child
-        link="${robot_name}_pan_link"/>
+        link="${robot_name}_pan_link" />
       <dynamics
         friction="0.1"
-        damping="0.1"/>
+        damping="0.1" />
     </joint>
     <link name="${robot_name}_pan_link">
@@ -22,20 +22,20 @@
         <origin
           rpy="0 0 ${pi/2}"
-          xyz="0 0 0"/>
+          xyz="0 0 0" />
         <geometry>
           <mesh
             filename="package://interbotix_xslocobot_descriptions/meshes/locobot_meshes/locobot_pan.stl"
-            scale="0.001 0.001 0.001"/>
-        </geometry>
-        <material name="interbotix_black"/>
+            scale="0.001 0.001 0.001" />
+        </geometry>
+        <material name="interbotix_black" />
       </visual>
       <collision>
         <origin
           rpy="0 0 ${pi/2}"
-          xyz="0 0 0"/>
+          xyz="0 0 0" />
         <geometry>
           <mesh
             filename="package://interbotix_xslocobot_descriptions/meshes/locobot_meshes/locobot_pan.stl"
-            scale="0.001 0.001 0.001"/>
+            scale="0.001 0.001 0.001" />
         </geometry>
       </collision>
@@ -43,6 +43,6 @@
         <origin
           rpy="0 0 ${pi/2}"
-          xyz="0.012 0.000496 0.018504"/>
-        <mass value="0.098997"/>
+          xyz="0.012 0.000496 0.018504" />
+        <mass value="0.098997" />
         <inertia
           ixx="0.0000276300"
@@ -51,5 +51,5 @@
           iyy="0.0000204300"
           iyz="-0.0000000421"
-          izz="0.0000276300"/>
+          izz="0.0000276300" />
       </inertial>
     </link>
@@ -59,20 +59,20 @@
     </gazebo>
     <joint name="tilt" type="revolute">
-      <axis xyz="0 1 0"/>
+      <axis xyz="0 1 0" />
       <limit
         effort="2"
         lower="${-pi/2}"
         upper="${radians(75)}"
-        velocity="${pi}"/>
+        velocity="${pi}" />
       <origin
-        rpy="0 0 0"
-        xyz="0.025034 0 0.019"/>
+        rpy="0 0.8 0"
+        xyz="0.025034 0 0.019" />
       <parent
-        link="${robot_name}_pan_link"/>
+        link="${robot_name}_pan_link" />
       <child
-        link="${robot_name}_tilt_link"/>
+        link="${robot_name}_tilt_link" />
       <dynamics
         friction="0.1"
-        damping="0.1"/>
+        damping="0.1" />
     </joint>
     <xacro:if value="${hardware_type == 'gz_classic'}">
@@ -86,5 +86,5 @@
             <param name="max">"${pi/2}"</param>
           </command_interface>
-          <state_interface name="position"/>
+          <state_interface name="position" />
         </joint>
         <joint name="tilt">
@@ -93,5 +93,5 @@
             <param name="max">"${radians(75)}"</param>
           </command_interface>
-          <state_interface name="position"/>
+          <state_interface name="position" />
         </joint>
       </ros2_control>
@@ -101,20 +101,20 @@
         <origin
           rpy="0 0 ${pi/2}"
-          xyz="0 0 0"/>
+          xyz="0 0 0" />
         <geometry>
           <mesh
             filename="package://interbotix_xslocobot_descriptions/meshes/locobot_meshes/locobot_tilt.stl"
-            scale="0.001 0.001 0.001"/>
-        </geometry>
-        <material name="interbotix_black"/>
+            scale="0.001 0.001 0.001" />
+        </geometry>
+        <material name="interbotix_black" />
       </visual>
       <collision>
         <origin
           rpy="0 0 ${pi/2}"
-          xyz="0 0 0"/>
+          xyz="0 0 0" />
         <geometry>
           <mesh
             filename="package://interbotix_xslocobot_descriptions/meshes/locobot_meshes/locobot_tilt.stl"
-            scale="0.001 0.001 0.001"/>
+            scale="0.001 0.001 0.001" />
         </geometry>
       </collision>
@@ -122,6 +122,6 @@
         <origin
           rpy="0 0 ${pi/2}"
-          xyz="0.0237737000 -0.0000016331 0.0000077432"/>
-        <mass value="0.019845"/>
+          xyz="0.0237737000 -0.0000016331 0.0000077432" />
+        <mass value="0.019845" />
         <inertia
           ixx="0.0000021677"
@@ -130,5 +130,5 @@
           iyy="0.0000063634"
           iyz="0.0000000003"
-          izz="0.0000066157"/>
+          izz="0.0000066157" />
       </inertial>
     </link>
@@ -140,9 +140,9 @@
       <origin
         rpy="0 0 0"
-        xyz="0.05318 0.0175 0.000009"/>
+        xyz="0.05318 0.0175 0.000009" />
       <parent
-        link="${robot_name}_tilt_link"/>
+        link="${robot_name}_tilt_link" />
       <child
-        link="camera_${robot_name}_link"/>
+        link="camera_${robot_name}_link" />
     </joint>
     <gazebo reference="camera">
@@ -153,13 +153,13 @@
         <origin
           rpy="0 0 0"
-          xyz="0 0 0"/>
+          xyz="0 0 0" />
         <geometry>
           <mesh
             filename="package://interbotix_xslocobot_descriptions/meshes/locobot_meshes/locobot_camera.stl"
-            scale="0.001 0.001 0.001"/>
+            scale="0.001 0.001 0.001" />
         </geometry>
         <material name="">
           <color
-            rgba="0.55 0.55 0.55 1"/>
+            rgba="0.55 0.55 0.55 1" />
         </material>
       </visual>
@@ -167,9 +167,9 @@
         <origin
           rpy="0 0 0"
-          xyz="0 0 0"/>
+          xyz="0 0 0" />
         <geometry>
           <mesh
             filename="package://interbotix_xslocobot_descriptions/meshes/locobot_meshes/locobot_camera.stl"
-            scale="0.001 0.001 0.001"/>
+            scale="0.001 0.001 0.001" />
         </geometry>
       </collision>
@@ -177,6 +177,6 @@
         <origin
           rpy="0 0 0"
-          xyz="-0.008972 -0.015818 0.000003"/>
-        <mass value="0.072"/>
+          xyz="-0.008972 -0.015818 0.000003" />
+        <mass value="0.072" />
         <inertia
           ixx="0.0000465400"
@@ -185,5 +185,5 @@
           iyy="0.0000069128"
           iyz="0.0000000248"
-          izz="0.0000468600"/>
+          izz="0.0000468600" />
       </inertial>
     </link>
@@ -195,17 +195,29 @@
     <!-- https://github.com/ros-simulation/gazebo_ros_pkgs/issues/243 -->
     <joint name="camera_depth_joint" type="fixed">
-      <origin rpy="${-pi/2} 0 ${-pi/2}" xyz="0 0 0"/>
-      <parent link="camera_${robot_name}_link"/>
-      <child link="${robot_name}_camera_depth_link"/>
+      <origin rpy="${-pi/2} 0 ${-pi/2}" xyz="0 0 0" />
+      <parent link="camera_${robot_name}_link" />
+      <child link="${robot_name}_camera_depth_link" />
     </joint>
     <link name="${robot_name}_camera_depth_link">
-      <origin rpy="0 0 0" xyz="0 0 0"/>
-    </link>
+      <origin rpy="0 0 0" xyz="0 0 0" />
+      <!-- <ignition_frame_id>${robot_name}_base_footprint</ignition_frame_id> -->
+    </link>
+    <!-- <joint name="depth_frame_to_link" type="fixed">
+      <origin rpy="0 0 0" xyz="0 0 0" />
+      <parent link="camera_${robot_name}_link" />
+      <child link="${robot_name}/camera_${robot_name}_link/rgbd_sensor" />
+    </joint>
+    <link name="${robot_name}/camera_${robot_name}_link/rgbd_sensor">
+      <origin rpy="0 0 0" xyz="0 0 0" />
+      <ignition_frame_id>/${robot_name}_base_footprint</ignition_frame_id>
+    </link> -->
     <gazebo reference="camera_${robot_name}_link">
-      <sensor name="camera_frame_sensor" type="depth">
+      <sensor name="rgbd_sensor" type="rgbd_camera">
+        <topic>/rgbd_camera</topic>
+        <ignition_frame_id>camera_${robot_name}_link</ignition_frame_id>
         <always_on>true</always_on>
-        <update_rate>30.0</update_rate>
-        <ignition_frame_id>${robot_name}_camera_depth_link</ignition_frame_id>
-        <camera>
+        <update_rate>1</update_rate>
+        <camera name="rgbd_camera">
+          <optical_frame_id>camera_${robot_name}_link</optical_frame_id>
           <horizontal_fov>0.994837</horizontal_fov>
           <image>
@@ -215,45 +227,60 @@
           </image>
           <clip>
-            <near>0.01</near>
-            <far>10</far>
+            <near>0.3</near>
+            <far>6</far>
           </clip>
+          <depth_camera>
+            <output>
+              sensor_msgs/msg/PointCloud2
+            </output>
+            <clip>
+              <near>0.3</near>
+              <far>6</far>
+            </clip>
+          </depth_camera>
+          <distortion>
+            <k1>0.00000001</k1>
+            <k2>0.00000001</k2>
+            <k3>0.00000001</k3>
+            <p1>0.00000001</p1>
+            <p2>0.00000001</p2>
+          </distortion>
+          <!-- <intrinsics>
+            <cx>0</cx>
+            <cy>0</cy>
+          </intrinsics>
+          <projection>
+            <fx>0</fx>
+            <fy>0</fy>
+          </projection> -->
         </camera>
         <xacro:if value="${hardware_type == 'gz_classic'}">
-        <plugin filename="libgazebo_ros_camera.so" name="camera_frame_controller">
-          <!-- <ros>
-            <namespace>/$(arg robot_name)</namespace>
-          </ros> -->
-          <alwaysOn>true</alwaysOn>
-          <updateRate>0.0</updateRate>
-          <cameraName>camera</cameraName>
-          <imageTopicName>color/image_raw</imageTopicName>
-          <cameraInfoTopicName>color/camera_info</cameraInfoTopicName>
-          <depthImageTopicName>aligned_depth_to_color/image_raw</depthImageTopicName>
-          <depthImageCameraInfoTopicName>aligned_depth_to_color/camera_info</depthImageCameraInfoTopicName>
-          <pointCloudTopicName>depth_registered/points</pointCloudTopicName>
-          <frameName>${robot_name}_camera_depth_link</frameName>
-          <pointCloudCutoff>0.01</pointCloudCutoff>
-          <pointCloudCutoffMax>10</pointCloudCutoffMax>
-          <distortionK1>0.00000001</distortionK1>
-          <distortionK2>0.00000001</distortionK2>
-          <distortionK3>0.00000001</distortionK3>
-          <distortionT1>0.00000001</distortionT1>
-          <distortionT2>0.00000001</distortionT2>
-          <CxPrime>0</CxPrime>
-          <Cx>0</Cx>
-          <Cy>0</Cy>
-          <focalLength>0</focalLength>
-          <hackBaseline>0</hackBaseline>
-        </plugin>
-      </xacro:if>
-      <!-- <xacro:if value="${hardware_type == 'gz_ignition'}">
-        <plugin
-            filename="RosGzPointCloud"
-            name="ros_gz_point_cloud::PointCloud">
-            <namespace>custom_params</namespace> -->
-            <!-- <topic>pc2</topic> -->
-            <!-- <frame_id>${robot_name}_camera_depth_link</frame_id>
+          <plugin filename="libgazebo_ros_camera.so" name="camera_frame_controller">
+            <ros>
+              <namespace>/$(arg robot_name)</namespace>
+            </ros>
+            <alwaysOn>true</alwaysOn>
+            <updateRate>0.0</updateRate>
+            <cameraName>camera</cameraName>
+            <imageTopicName>color/image_raw</imageTopicName>
+            <cameraInfoTopicName>color/camera_info</cameraInfoTopicName>
+            <depthImageTopicName>aligned_depth_to_color/image_raw</depthImageTopicName>
+            <depthImageCameraInfoTopicName>aligned_depth_to_color/camera_info</depthImageCameraInfoTopicName>
+            <pointCloudTopicName>depth_registered/points</pointCloudTopicName>
+            <frameName>${robot_name}_camera_depth_link</frameName>
+            <pointCloudCutoff>0.01</pointCloudCutoff>
+            <pointCloudCutoffMax>10</pointCloudCutoffMax>
+            <distortionK1>0.00000001</distortionK1>
+            <distortionK2>0.00000001</distortionK2>
+            <distortionK3>0.00000001</distortionK3>
+            <distortionT1>0.00000001</distortionT1>
+            <distortionT2>0.00000001</distortionT2>
+            <CxPrime>0</CxPrime>
+            <Cx>0</Cx>
+            <Cy>0</Cy>
+            <focalLength>0</focalLength>
+            <hackBaseline>0</hackBaseline>
           </plugin>
-      </xacro:if> -->
+        </xacro:if>
       </sensor>
     </gazebo>
