Commit message: reorg

File: interbotix_ros_xslocobots/interbotix_xslocobot_descriptions/urdf/arms/mobile_wx250s.urdf.xacro (robot description, xacro)
@@ -9,6 +9,6 @@
   <xacro:property name="hardware_type" value="$(arg hardware_type)" />
   <xacro:property name="pi_offset" value="0.00001" />
-  <!-- <xacro:include filename="$(find
-  interbotix_xslocobot_descriptions)/urdf/arms/arm_control.urdf.xacro"/> -->
+  <xacro:property name="initial_positions_file" default="$(find interbotix_xslocobot_sim)/config/initial_positions.yaml" />
+  <xacro:property name="initial_positions" default="${xacro.load_yaml(initial_positions_file)}" />
   <xacro:include filename="$(find interbotix_xslocobot_descriptions)/urdf/arms/ar_tag.urdf.xacro" />
   <link name="${robot_name}_arm_base_link">
@@ -56,5 +56,5 @@
       velocity="${waist_limit_vel}" />
     <origin
-      rpy="0 0 0"
+      rpy="0 0 ${initial_positions['waist']}"
       xyz="0 0 0.066175" />
     <parent
@@ -110,5 +110,5 @@
       velocity="${shoulder_limit_vel}" />
     <origin
-      rpy="0 0 0"
+      rpy="0 ${initial_positions['shoulder']} 0"
       xyz="0 0 0.03865" />
     <parent
@@ -164,5 +164,5 @@
       velocity="${elbow_limit_vel}" />
     <origin
-      rpy="0 0 0"
+      rpy="0 ${initial_positions['elbow']} 0"
       xyz="0.04975 0 0.25" />
     <parent
@@ -217,5 +217,5 @@
       upper="${forearm_roll_limit_upper}"
       velocity="${forearm_roll_limit_vel}" />
-    <origin rpy="0 0 0" xyz="0.175 0 0" />
+    <origin rpy="${initial_positions['forearm_roll']} 0 0" xyz="0.175 0 0" />
     <parent
       link="${robot_name}_upper_forearm_link" />
@@ -270,5 +270,5 @@
       velocity="${wrist_angle_limit_vel}" />
     <origin
-      rpy="0 0 0"
+      rpy="0  ${initial_positions['wrist_angle']} 0"
       xyz="0.075 0 0" />
     <parent
@@ -326,5 +326,5 @@
         velocity="${wrist_rotate_limit_vel}" />
       <origin
-        rpy="0 0 0"
+        rpy="${initial_positions['wrist_rotate']} 0 0"
         xyz="0.065 0 0" />
       <parent
@@ -525,5 +525,5 @@
           <origin
             rpy="0 0 0"
-            xyz="0 0 0" />
+            xyz="0 ${initial_positions['left_finger']} 0" />
           <parent
             link="${robot_name}_fingers_link" />
@@ -578,5 +578,5 @@
           <origin
             rpy="0 0 0"
-            xyz="0 0 0" />
+            xyz="0  ${initial_positions['right_finger']} 0" />
           <parent
             link="${robot_name}_fingers_link" />
@@ -651,4 +651,148 @@
           </inertial>
         </link>
+        <gazebo reference="${robot_name}_ar_tag_link">
+          <visual>
+            <material>
+              <xacro:include
+                filename="$(find interbotix_xslocobot_descriptions)/urdf/colors.urdf.xacro" />
+              <xacro:color color="black" />
+            </material>
+          </visual>
+        </gazebo>
+        <gazebo reference="{robot_name}_arm_base_link">
+          <visual>
+            <material>
+              <xacro:include
+                filename="$(find interbotix_xslocobot_descriptions)/urdf/colors.urdf.xacro" />
+              <xacro:color color="black" />
+            </material>
+          </visual>
+        </gazebo>
+        <gazebo reference="${robot_name}_shoulder_link">
+          <visual>
+            <material>
+              <xacro:include
+                filename="$(find interbotix_xslocobot_descriptions)/urdf/colors.urdf.xacro" />
+              <xacro:color color="black" />
+            </material>
+          </visual>
+        </gazebo>
+        <gazebo reference="${robot_name}_upper_arm_link">
+          <visual>
+            <material>
+              <xacro:include
+                filename="$(find interbotix_xslocobot_descriptions)/urdf/colors.urdf.xacro" />
+              <xacro:color color="black" />
+            </material>
+          </visual>
+        </gazebo>
+        <gazebo reference="${robot_name}_upper_forearm_link">
+          <visual>
+            <material>
+              <xacro:include
+                filename="$(find interbotix_xslocobot_descriptions)/urdf/colors.urdf.xacro" />
+              <xacro:color color="black" />
+            </material>
+          </visual>
+        </gazebo>
+        <gazebo reference="${robot_name}_lower_forearm_link">
+          <visual>
+            <material>
+              <xacro:include
+                filename="$(find interbotix_xslocobot_descriptions)/urdf/colors.urdf.xacro" />
+              <xacro:color color="black" />
+            </material>
+          </visual>
+        </gazebo>
+        <gazebo reference="${robot_name}_wrist_link">
+          <visual>
+            <material>
+              <xacro:include
+                filename="$(find interbotix_xslocobot_descriptions)/urdf/colors.urdf.xacro" />
+              <xacro:color color="black" />
+            </material>
+          </visual>
+        </gazebo>
+        <gazebo reference="${robot_name}_gripper_link">
+          <visual>
+            <material>
+              <xacro:include
+                filename="$(find interbotix_xslocobot_descriptions)/urdf/colors.urdf.xacro" />
+              <xacro:color color="black" />
+            </material>
+          </visual>
+        </gazebo>
+        <gazebo reference="${robot_name}_gripper_prop_link">
+          <visual>
+            <material>
+              <xacro:include
+                filename="$(find interbotix_xslocobot_descriptions)/urdf/colors.urdf.xacro" />
+              <xacro:color color="black" />
+            </material>
+          </visual>
+        </gazebo>
+        <gazebo reference="${robot_name}_ee_arm_link">
+          <visual>
+            <material>
+              <xacro:include
+                filename="$(find interbotix_xslocobot_descriptions)/urdf/colors.urdf.xacro" />
+              <xacro:color color="black" />
+            </material>
+          </visual>
+        </gazebo>
+        <gazebo reference="${robot_name}_fingers_link">
+          <visual>
+            <material>
+              <xacro:include
+                filename="$(find interbotix_xslocobot_descriptions)/urdf/colors.urdf.xacro" />
+              <xacro:color color="black" />
+            </material>
+          </visual>
+        </gazebo>
+        <gazebo reference="${robot_name}_ee_gripper_link">
+          <visual>
+            <material>
+              <xacro:include
+                filename="$(find interbotix_xslocobot_descriptions)/urdf/colors.urdf.xacro" />
+              <xacro:color color="black" />
+            </material>
+          </visual>
+        </gazebo>
+        <gazebo reference="${robot_name}_gripper_link">
+          <visual>
+            <material>
+              <xacro:include
+                filename="$(find interbotix_xslocobot_descriptions)/urdf/colors.urdf.xacro" />
+              <xacro:color color="black" />
+            </material>
+          </visual>
+        </gazebo>
+        <gazebo reference="${robot_name}_gripper_bar_link">
+          <visual>
+            <material>
+              <xacro:include
+                filename="$(find interbotix_xslocobot_descriptions)/urdf/colors.urdf.xacro" />
+              <xacro:color color="black" />
+            </material>
+          </visual>
+        </gazebo>
+        <gazebo reference="${robot_name}_left_finger_link">
+          <visual>
+            <material>
+              <xacro:include
+                filename="$(find interbotix_xslocobot_descriptions)/urdf/colors.urdf.xacro" />
+              <xacro:color color="black" />
+            </material>
+          </visual>
+        </gazebo>
+        <gazebo reference="${robot_name}_right_finger_link">
+          <visual>
+            <material>
+              <xacro:include
+                filename="$(find interbotix_xslocobot_descriptions)/urdf/colors.urdf.xacro" />
+              <xacro:color color="black" />
+            </material>
+          </visual>
+        </gazebo>
       </xacro:if> <!--
       show_gripper_fingers -->

File: interbotix_ros_xslocobots/interbotix_xslocobot_descriptions/urdf/base/kobuki/locobot_kobuki.urdf.xacro (robot description, xacro)
@@ -38,5 +38,11 @@
     # POSSIBILITY OF SUCH DAMAGE.
   -->
-  <link name="${robot_name}_base_footprint"/>
+  <!-- <link name="world" />
+  <joint name="virtual_joint" type="planar">
+    <parent link="world" />
+    <child
+      link="${robot_name}_base_footprint" />
+  </joint> -->
+  <link name="${robot_name}_base_footprint" />
   <joint name="base_joint" type="fixed">
     <origin

File: interbotix_ros_xslocobots/interbotix_xslocobot_descriptions/urdf/body/pan_and_tilt.urdf.xacro (robot description, xacro)
@@ -1,4 +1,6 @@
 <?xml version="1.0"?>
 <robot xmlns:xacro="http://ros.org/wiki/xacro">
+  <xacro:property name="initial_positions_file" default="$(find interbotix_xslocobot_sim)/config/initial_positions.yaml" />
+  <xacro:property name="initial_positions" default="${xacro.load_yaml(initial_positions_file)}" />
   <xacro:macro name="pan_and_tilt" params="*origin">
     <joint name="pan" type="revolute">
@@ -66,5 +68,5 @@
         velocity="${pi}" />
       <origin
-        rpy="0 0.8 0"
+        rpy="0 ${initial_positions['tilt']} 0"
         xyz="0.025034 0 0.019" />
       <parent
@@ -213,9 +215,28 @@
     </link> -->
     <gazebo reference="camera_${robot_name}_link">
+      <sensor name="camera" type="camera">
+        <topic>/camera</topic>
+        <ignition_frame_id>camera_${robot_name}_link</ignition_frame_id>
+        <always_on>true</always_on>
+        <update_rate>5</update_rate>
+        <topic>camera</topic>
+        <camera>
+          <optical_frame_id>camera_${robot_name}_link</optical_frame_id>
+          <horizontal_fov>0.994837</horizontal_fov>
+            <image>
+                <width>640</width>
+                <height>480</height>
+            </image>
+            <clip>
+                <near>0.01</near>
+                <far>6</far>
+            </clip>
+        </camera>
+      </sensor>
       <sensor name="rgbd_sensor" type="rgbd_camera">
         <topic>/rgbd_camera</topic>
         <ignition_frame_id>camera_${robot_name}_link</ignition_frame_id>
         <always_on>true</always_on>
-        <update_rate>30</update_rate>
+        <update_rate>5</update_rate>
         <camera name="rgbd_camera">
           <optical_frame_id>camera_${robot_name}_link</optical_frame_id>

File: interbotix_ros_xslocobots/interbotix_xslocobot_descriptions/urdf/control.urdf.xacro (robot description, xacro)
@@ -1,5 +1,5 @@
 <?xml version="1.0"?>
 <robot xmlns:xacro="http://ros.org/wiki/xacro">
-  <xacro:macro name="hardware_interface">
+  <xacro:macro name="hardware_interface" params="initial_positions">
     <hardware>
       <!-- If we are using the actual, physical robot -->
@@ -26,52 +26,52 @@
     <joint name="waist">
       <command_interface name="position">
-        <param name="min">"${waist_limit_lower}"</param>
-        <param name="max">"${waist_limit_upper}"</param>
+        <param name="min">${waist_limit_lower}</param>
+        <param name="max">${waist_limit_upper}</param>
       </command_interface>
       <state_interface name="position" />
-      <param name="initial_position">0.00</param>
+      <param name="initial_position">${initial_positions['waist']}</param>
     </joint>
     <joint name="shoulder">
       <command_interface name="position">
-        <param name="min">"${shoulder_limit_lower}"</param>
-        <param name="max">"${shoulder_limit_upper}"</param>
+        <param name="min">${shoulder_limit_lower}</param>
+        <param name="max">${shoulder_limit_upper}</param>
       </command_interface>
       <state_interface name="position" />
-      <param name="initial_position">0.00</param>
+      <param name="initial_position">${initial_positions['shoulder']}</param>
     </joint>
     <joint name="elbow">
       <command_interface name="position">
-        <param name="min">"${elbow_limit_lower}"</param>
-        <param name="max">"${elbow_limit_upper}"</param>
+        <param name="min">${elbow_limit_lower}</param>
+        <param name="max">${elbow_limit_upper}</param>
       </command_interface>
       <state_interface name="position" />
-      <param name="initial_position">0.00</param>
+      <param name="initial_position">${initial_positions['elbow']}</param>
     </joint>
     <xacro:if value="${dof >= 6}">
       <joint name="forearm_roll">
         <command_interface name="position">
-          <param name="min">"${forearm_roll_limit_lower}"</param>
-          <param name="max">"${forearm_roll_limit_upper}"</param>
+          <param name="min">${forearm_roll_limit_lower}</param>
+          <param name="max">${forearm_roll_limit_upper}</param>
         </command_interface>
         <state_interface name="position" />
-        <param name="initial_position">0.00</param>
+        <param name="initial_position">${initial_positions['forearm_roll']}</param>
       </joint>
     </xacro:if>
     <joint name="wrist_angle">
       <command_interface name="position">
-        <param name="min">"${wrist_angle_limit_lower}"</param>
-        <param name="max">"${wrist_angle_limit_upper}"</param>
+        <param name="min">${wrist_angle_limit_lower}</param>
+        <param name="max">${wrist_angle_limit_upper}</param>
       </command_interface>
       <state_interface name="position" />
-      <param name="initial_position">0.00</param>
+      <param name="initial_position">${initial_positions['wrist_angle']}</param>
     </joint>
     <xacro:if value="${dof >= 5}">
       <joint name="wrist_rotate">
         <command_interface name="position">
-          <param name="min">"${wrist_rotate_limit_lower}"</param>
-          <param name="max">"${wrist_rotate_limit_upper}"</param>
+          <param name="min">${wrist_rotate_limit_lower}</param>
+          <param name="max">${wrist_rotate_limit_upper}</param>
         </command_interface>
         <state_interface name="position" />
-        <param name="initial_position">0.00</param>
+        <param name="initial_position">${initial_positions['wrist_rotate']}</param>
       </joint>
     </xacro:if>
@@ -90,5 +90,5 @@
           </command_interface>
           <state_interface name="position" />
-          <param name="initial_position">0.0195</param>
+          <param name="initial_position">${initial_positions['left_finger']}</param>
         </joint>
         <xacro:if value="${hardware_type in ('gz_classic', 'gz_ignition')}">
@@ -98,8 +98,8 @@
             <command_interface name="position">
               <param name="min">${-finger_limit_upper}</param>
-              <param name="max">${-finger_limit_lower}"</param>
+              <param name="max">${-finger_limit_lower}</param>
             </command_interface>
             <state_interface name="position" />
-            <param name="initial_position">-0.0195</param>
+            <param name="initial_position">${initial_positions['right_finger']}</param>
           </joint>
         </xacro:if>
@@ -109,10 +109,12 @@
       <command_interface name="position" />
       <state_interface name="position" />
-      <param name="initial_position">0.0</param>  <!-- initial position for the GenericSystem -->
+      <param name="initial_position">${initial_positions['pan']}</param>  <!-- initial position for
+      the GenericSystem -->
     </joint>
     <joint name="tilt">
       <command_interface name="position" />
       <state_interface name="position" />
-      <param name="initial_position">0.0</param>  <!-- initial position for the GenericSystem -->
+      <param name="initial_position">${initial_positions['tilt']}</param>  <!-- initial position for
+      the GenericSystem -->
     </joint>
     <xacro:if value="${base_type == 'create3'}">

File: interbotix_ros_xslocobots/interbotix_xslocobot_descriptions/urdf/locobot.urdf.xacro (robot description, xacro)
@@ -49,4 +49,8 @@
   <!-- <xacro:property name="right_finger_limit_upper" value="0.01" /> -->
   <xacro:property name="finger_limit_vel" value="1.0" />
+  <xacro:arg name="initial_positions_file"
+    default="$(find interbotix_xslocobot_sim)/config/initial_positions.yaml" />
+  <xacro:property name="initial_positions_file" default="$(arg initial_positions_file)" />
+  <xacro:property name="initial_positions" default="${xacro.load_yaml(initial_positions_file)}" />
   <xacro:if value="${urdf_loc != ''}">
     <xacro:include filename="${urdf_loc}" />
@@ -56,10 +60,10 @@
       filename="package://interbotix_common_sim/media/materials/textures/interbotix_black.png" />
   </material>
-  <xacro:include filename="$(find interbotix_xslocobot_descriptions)/urdf/plate.urdf.xacro" />
+  <xacro:include filename="$(find interbotix_xslocobot_descriptions)/urdf/body/plate.urdf.xacro" />
   <xacro:include filename="$(find interbotix_xslocobot_descriptions)/urdf/lidar.urdf.xacro" />
-  <xacro:include filename="$(find interbotix_xslocobot_descriptions)/urdf/battery.urdf.xacro" />
-  <xacro:include filename="$(find interbotix_xslocobot_descriptions)/urdf/arm_cradle.urdf.xacro" />
-  <xacro:include filename="$(find interbotix_xslocobot_descriptions)/urdf/camera_tower.urdf.xacro" />
-  <xacro:include filename="$(find interbotix_xslocobot_descriptions)/urdf/pan_and_tilt.urdf.xacro" />
+  <xacro:include filename="$(find interbotix_xslocobot_descriptions)/urdf/body/battery.urdf.xacro" />
+  <xacro:include filename="$(find interbotix_xslocobot_descriptions)/urdf/body/arm_cradle.urdf.xacro" />
+  <xacro:include filename="$(find interbotix_xslocobot_descriptions)/urdf/body/camera_tower.urdf.xacro" />
+  <xacro:include filename="$(find interbotix_xslocobot_descriptions)/urdf/body/pan_and_tilt.urdf.xacro" />
   <xacro:if value="${arm_type == 'mobile_wx250s'}">
     <xacro:property name="camera_tower_size" value="large" />
@@ -70,10 +74,10 @@
   <xacro:if value="${base_type == 'kobuki'}">
     <xacro:include
-      filename="$(find interbotix_xslocobot_descriptions)/urdf/kobuki_version/locobot_kobuki.urdf.xacro" />
+      filename="$(find interbotix_xslocobot_descriptions)/urdf/base/kobuki/locobot_kobuki.urdf.xacro" />
     <xacro:property name="mesh_scale" value="0.001 0.001 0.001" />
   </xacro:if> <!-- kobuki -->
   <xacro:if value="${base_type == 'create3'}">
     <xacro:include
-      filename="$(find interbotix_xslocobot_descriptions)/urdf/create3_version/locobot_create3.urdf.xacro" />
+      filename="$(find interbotix_xslocobot_descriptions)/urdf/base/create3/locobot_create3.urdf.xacro" />
     <xacro:property name="mesh_scale" value="1 1 1" />
   </xacro:if> <!-- create3 -->
@@ -258,5 +262,5 @@
       <xacro:pan_and_tilt>
         <origin
-          rpy="0 0 0"
+          rpy="0 0 ${initial_positions['pan']}"
           xyz="0.047228 0 0.44425" />
       </xacro:pan_and_tilt>
@@ -358,5 +362,5 @@
   <!-- Defines hardware interface. -->
   <ros2_control name="SystemControl" type="system">
-    <xacro:hardware_interface />
+    <xacro:hardware_interface initial_positions="${initial_positions}" />
     <!-- TODO:(speralta): Move pan_and_tilt sensors here? -->
   </ros2_control>

File: interbotix_ros_xslocobots/interbotix_xslocobot_moveit/config/srdf/locobot_wx250s.srdf.xacro (robot description, xacro)
@@ -35,5 +35,5 @@
     </group>
     <!--GROUP STATES - Purpose - Define a named state for a particular group, in terms of joint values. This is useful to define states like 'folded arms'-->
-    <group_state name="Home" group="interbotix_arm">
+    <group_state name="Sleep" group="interbotix_arm">
         <joint name="elbow" value="0" />
         <joint name="forearm_roll" value="0" />
@@ -43,5 +43,5 @@
         <joint name="wrist_rotate" value="0" />
     </group_state>
-    <group_state name="Sleep" group="interbotix_arm">
+    <!-- <group_state name="Sleep" group="interbotix_arm">
         <joint name="elbow" value="1.55" />
         <joint name="forearm_roll" value="0" />
@@ -50,5 +50,5 @@
         <joint name="wrist_angle" value="0.5" />
         <joint name="wrist_rotate" value="0" />
-    </group_state>
+    </group_state> -->
     <group_state name="Upright" group="interbotix_arm">
         <joint name="elbow" value="-1.5708" />
@@ -72,5 +72,5 @@
     </group_state>
     <!-- Define how the robot moves in its environment, i.e., connection to robot's root link -->
-    <virtual_joint name="virtual_joint" type="planar" parent_frame="odom"
+    <virtual_joint name="virtual_joint" type="planar" parent_frame="world"
         child_link="locobot_base_footprint" /> <!-- type can be planar, floating or fixed -->
     <!--END EFFECTOR - Purpose - Represent information about an end effector.-->
