Commit message: waist lateral position

File: interbotix_ros_xslocobots/interbotix_xslocobot_descriptions/urdf/arms/ar_tag.urdf.xacro (robot description, xacro)
@@ -55,4 +55,57 @@
       <material>Gazebo/DarkGrey</material>
     </gazebo>
+      <joint name="arm_base_camera_link" type="fixed">
+        <origin rpy="0 0.025 0" xyz="0.005 0 0" />
+        <parent link="${robot_name}_ar_tag_link" />
+        <child link="${robot_name}_arm_base_camera_link" />
+      </joint>
+      <link name="${robot_name}_arm_base_camera_link">
+        <!-- <origin rpy="0 0 0" xyz="0.02 0 0.02" /> -->
+        <ignition_frame_id>/${robot_name}_arm_base_camera_link</ignition_frame_id>
+        <!-- <collision>
+          <geometry>
+            <box size="0.01 0.02 0.03" />
+          </geometry>
+        </collision>
+        <visual>
+          <origin
+            rpy="0 0 0"
+            xyz="0 0 0" />
+          <geometry>
+            <box size="0.01 0.02 0.03" />
+          </geometry>
+          <material name="interbotix_black" />
+        </visual> -->
+      </link>
+    <!-- <gazebo reference="${robot_name}_arm_base_camera_link">
+      <material>Gazebo/Darkblack</material>
+        <sensor name="camera_arm_base" type="camera">
+          <topic>/camera_arm_base</topic>
+          <ignition_frame_id>${robot_name}_arm_base_camera_link</ignition_frame_id>
+          <always_on>true</always_on>
+          <update_rate>5</update_rate>
+          <camera name="camera_arm_base">
+            <optical_frame_id>${robot_name}_arm_base_camera_link</optical_frame_id>
+            <horizontal_fov>0.994837</horizontal_fov>
+            <update_rate>10</update_rate>
+            <image>
+              <format>R8G8B8</format>
+              <width>640</width>
+              <height>480</height>
+            </image>
+            <clip>
+              <near>0.01</near>
+              <far>6</far>
+            </clip>
+            <distortion>
+              <k1>0.00000001</k1>
+              <k2>0.00000001</k2>
+              <k3>0.00000001</k3>
+              <p1>0.00000001</p1>
+              <p2>0.00000001</p2>
+            </distortion>
+     </camera>
+        </sensor>
+    </gazebo> -->
   </xacro:if> <!-- show_ar_tag -->
 </robot>

File: interbotix_ros_xslocobots/interbotix_xslocobot_descriptions/urdf/arms/mobile_wx250s.urdf.xacro (robot description, xacro)
@@ -48,4 +48,52 @@
     </inertial>
   </link>
+<!--
+    <joint name="arm_base_camera_link" type="fixed">
+      <origin rpy="0 0.6 0" xyz="-0.05 0 0.5" />
+      <parent link="${robot_name}_arm_base_link" />
+      <child link="${robot_name}_arm_base_camera_link" />
+    </joint>
+    <link name="${robot_name}_arm_base_camera_link">
+      <origin rpy="0 0 0" xyz="0 0 0" />
+      <ignition_frame_id>/${robot_name}_arm_base_camera_link</ignition_frame_id>
+    </link>
+  <gazebo reference="${robot_name}_arm_base_camera_link">
+    <material>Gazebo/Darkblack</material>
+      <sensor name="camera_arm_base" type="camera">
+        <topic>/camera_arm_base</topic>
+        <ignition_frame_id>${robot_name}_arm_base_camera_link</ignition_frame_id>
+        <always_on>true</always_on>
+        <update_rate>5</update_rate>
+        <camera name="camera_arm_base">
+          <optical_frame_id>${robot_name}_arm_base_camera_link</optical_frame_id>
+          <horizontal_fov>0.994837</horizontal_fov>
+          <update_rate>10</update_rate>
+          <image>
+            <format>R8G8B8</format>
+            <width>640</width>
+            <height>480</height>
+          </image>
+          <clip>
+            <near>0.01</near>
+            <far>6</far>
+          </clip>
+          <distortion>
+            <k1>0.00000001</k1>
+            <k2>0.00000001</k2>
+            <k3>0.00000001</k3>
+            <p1>0.00000001</p1>
+            <p2>0.00000001</p2>
+          </distortion> -->
+          <!-- <intrinsics>
+            <cx>0</cx>
+            <cy>0</cy>
+          </intrinsics>
+          <projection>
+            <fx>0</fx>
+            <fy>0</fy>
+          </projection> -->
+        <!-- </camera>
+      </sensor>
+  </gazebo> -->
   <joint name="waist" type="revolute">
     <axis xyz="0 0 1" />
@@ -57,5 +105,5 @@
     <origin
       rpy="0 0 ${initial_positions['waist']}"
-      xyz="0 0 0.066175" />
+      xyz="0 ${initial_positions['waist_lateral_position']} 0.066175" />
     <parent
       link="${robot_name}_arm_base_link" />

File: interbotix_ros_xslocobots/interbotix_xslocobot_descriptions/urdf/body/pan_and_tilt.urdf.xacro (robot description, xacro)
@@ -220,16 +220,32 @@
         <always_on>true</always_on>
         <update_rate>5</update_rate>
-        <topic>camera</topic>
-        <camera>
+        <camera name="camera">
           <optical_frame_id>camera_${robot_name}_link</optical_frame_id>
           <horizontal_fov>0.994837</horizontal_fov>
-            <image>
-                <width>640</width>
-                <height>480</height>
-            </image>
-            <clip>
-                <near>0.01</near>
-                <far>6</far>
-            </clip>
+          <update_rate>10</update_rate>
+          <image>
+            <format>R8G8B8</format>
+            <width>640</width>
+            <height>480</height>
+          </image>
+          <clip>
+            <near>0.01</near>
+            <far>6</far>
+          </clip>
+          <distortion>
+            <k1>0.00000001</k1>
+            <k2>0.00000001</k2>
+            <k3>0.00000001</k3>
+            <p1>0.00000001</p1>
+            <p2>0.00000001</p2>
+          </distortion>
+          <!-- <intrinsics>
+            <cx>0</cx>
+            <cy>0</cy>
+          </intrinsics>
+          <projection>
+            <fx>0</fx>
+            <fy>0</fy>
+          </projection> -->
         </camera>
       </sensor>
@@ -238,5 +254,5 @@
         <ignition_frame_id>camera_${robot_name}_link</ignition_frame_id>
         <always_on>true</always_on>
-        <update_rate>5</update_rate>
+        <update_rate>10</update_rate>
         <camera name="rgbd_camera">
           <optical_frame_id>camera_${robot_name}_link</optical_frame_id>
